File: 01_KiCad project/Nvum_CNC_expander.kicad_pcb (KiCad board)
At the start: 2 copper layers, 91 parts, among them J1 Conn_01x02_Female, J10 Conn_01x02_Female, J11 PS 14-24V, J12 Conn_01x10_Male, J2 Conn_01x02_Female, J3 Conn_01x02_Female, J4 Conn_01x02_Female, J5 Conn_01x02_Female, J6 Conn_01x02_Female, J7 Conn_01x02_Female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

Commit message: Add files via upload
Parts:
- added D21: 1.3W24V, Diode_THT:D_A-405_P12.70mm_Horizontal, F.Cu at (55.6, 72.4)
Other:
- board outline added: 105.4 x 69.8 mm
