File: 01_KiCad project/Nvum_CNC_expander.sch (KiCad schematic (older format))
At the start: 91 parts, among them J1 Conn_01x02_Female, J10 Conn_01x02_Female, J11 PS 14-24V, J12 Conn_01x10_Male, J2 Conn_01x02_Female, J3 Conn_01x02_Female, J4 Conn_01x02_Female, J5 Conn_01x02_Female, J6 Conn_01x02_Female, J7 Conn_01x02_Female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

Commit message: Add files via upload
Parts:
- added D21: 1.3W24V, Diode_THT:D_A-405_P12.70mm_Horizontal, symbol Device:D_Zener
Connections:
- net +24V: now also D21.1 (K)
- net GNDD: now also D21.2 (A)
Other:
- moved on the sheet: R41
Changed lines of the file:
@@
 L Device:R R41
 U 1 1 605D3CF3
-P 2400 8400
-F 0 "R41" H 2330 8354 50  0000 R CNN
-F 1 "100k" H 2330 8445 50  0000 R CNN
-F 2 "Resistor_SMD:R_0805_2012Metric_Pad1.20x1.40mm_HandSolder" V 2285 8400 50  0001 C CNN
-F 3 "~" H 2400 8400 50  0001 C CNN
-F 4 "power supply" H 2400 8400 50  0001 C CNN "Module"
-	1    2400 8400
+P 2550 8400
+F 0 "R41" H 2480 8354 50  0000 R CNN
+F 1 "100k" H 2480 8445 50  0000 R CNN
+F 2 "Resistor_SMD:R_0805_2012Metric_Pad1.20x1.40mm_HandSolder" V 2435 8400 50  0001 C CNN
+F 3 "~" H 2550 8400 50  0001 C CNN
+F 4 "power supply" H 2550 8400 50  0001 C CNN "Module"
+	1    2550 8400
 	0    -1   -1   0
 $EndComp
 Wire Wire Line
-	2550 8400 2750 8400
+	2700 8400 2750 8400
 Wire Wire Line
-	2250 8400 2100 8400
+	2400 8400 2100 8400
 Wire Wire Line
 	2100 8400 2100 8300
@@
 Wire Notes Line
 	3000 7700 3000 8000
+$Comp
+L Device:D_Zener D21
+U 1 1 60531878
+P 2100 8550
+F 0 "D21" V 2054 8630 50  0000 L CNN
+F 1 "1.3W24V" V 2145 8630 50  0000 L CNN
+F 2 "Diode_THT:D_A-405_P12.70mm_Horizontal" H 2100 8550 50  0001 C CNN
+F 3 "~" H 2100 8550 50  0001 C CNN
+	1    2100 8550
+	0    1    1    0
+$EndComp
+Connection ~ 2100 8400
+$Comp
+L power:GNDD #PWR0138
+U 1 1 6053DDB0
+P 2100 8750
+F 0 "#PWR0138" H 2100 8500 50  0001 C CNN
+F 1 "GNDD" H 2104 8595 50  0000 C CNN
+F 2 "" H 2100 8750 50  0001 C CNN
+F 3 "" H 2100 8750 50  0001 C CNN
+	1    2100 8750
+	1    0    0    -1
+$EndComp
+Wire Wire Line
+	2100 8750 2100 8700
 $EndSCHEMATC
